Commit message: add odom control

File: catkin_ws/src/sim/duckiebot_description/urdf/duckiebot.xacro (robot description, xacro)
@@ -1,3 +1,3 @@
-<?xml version='1.0'?>
+<?xml version='1.0' encoding="utf-8"?>
 <robot name="duckiebot" xmlns:xacro="http://www.ros.org/wiki/xacro">
   <xacro:property name="cameraSize" value="0.01"/>

File: catkin_ws/src/sim/mybot_description/urdf/mybot.xacro (robot description, xacro)
@@ -6,4 +6,23 @@
   <xacro:include filename="$(find mybot_description)/urdf/materials.xacro" />
   <xacro:include filename="$(find mybot_description)/urdf/macros.xacro" />
+  <!-- define inertias -->
+  <macro name="cylinder_inertia" params="m r h">
+    <inertia  ixx="${m*(3*r*r+h*h)/12}" ixy = "0" ixz = "0"
+      iyy="${m*(3*r*r+h*h)/12}" iyz = "0"
+      izz="${m*r*r/2}"
+    />
+  </macro>
+  <macro name="box_inertia" params="m x y z">
+    <inertia  ixx="${m*(y*y+z*z)/12}" ixy = "0" ixz = "0"
+      iyy="${m*(x*x+z*z)/12}" iyz = "0"
+      izz="${m*(x*x+z*z)/12}"
+    />
+  </macro>
+  <macro name="sphere_inertia" params="m r">
+    <inertia  ixx="${2*m*r*r/5}" ixy = "0" ixz = "0"
+      iyy="${2*m*r*r/5}" iyz = "0"
+      izz="${2*m*r*r/5}"
+    />
+  </macro>
   <link name='chassis'>
     <pose>0 0 0.1 0 0 0</pose>
@@ -12,13 +31,14 @@
       <mass value="30.0"/>
       <origin xyz="0.0 0 0.1" rpy=" 0 0 0"/>
-      <inertia
+      <box_inertia m="0.1" x="0.4" y="0.4" z="0.1" />
+      <!--<inertia
           ixx="0.1" ixy="0" ixz="0"
           iyy="0.1" iyz="0"
           izz="0.1"
-      />
+      />-->
     </inertial>
     <collision name='collision'>
       <geometry>
-        <box size=".4 .2 .1"/>
+        <box size=".4 .4 .1"/>
       </geometry>
     </collision>
@@ -26,5 +46,5 @@
       <origin xyz="0 0 0" rpy=" 0 0 0"/>
       <geometry>
-        <box size=".4 .2 .1"/>
+        <box size=".4 .4 .1"/>
       </geometry>
     </visual>
